Commit message: feature: real robot contorller(sine_wave base)

File: src/my_manipulator_description/urdf/my_robot.xacro (robot description, xacro)
@@ -21,9 +21,9 @@
     <parent link="base_link"/>
     <child link="articulation1"/>
-    <origin xyz="0 0 0.045" rpy="0 0 0"/>
+    <origin xyz="0 0 0.045" rpy="0 0 -1.57"/>
     <!-- 회전축 -->
     <axis xyz="0 0 1"/>
     <!-- 임시 limit -->
-    <limit lower="-1.57" upper="1.57" effort="1" velocity="1"/>
+    <limit lower="0" upper="3.14" effort="1" velocity="1"/>
   </joint>
   <!-- link1 -->
@@ -39,9 +39,9 @@
     <parent link="articulation1"/>
     <child link="link1"/>
-    <origin xyz="0 0.026 0.03" rpy="0 0 0"/>
+    <origin xyz="0 0.026 0.03" rpy="0 -1.57 0"/>
     <!-- 회전축 -->
     <axis xyz="0 1 0"/>
     <!-- 임시 limit -->
-    <limit lower="-1.57" upper="1.57" effort="1" velocity="1"/>
+    <limit lower="0" upper="3.14" effort="1" velocity="1"/>
   </joint>
   <!-- link2 -->
@@ -53,5 +53,5 @@
     </visual>
   </link>
-  <!-- joint2: link1 -> link2 -->
+  <!-- joint3: link1 -> link2 -->
   <joint name="joint3" type="revolute">
     <parent link="link1"/>
@@ -59,7 +59,7 @@
     <origin xyz="0 -0.046 0.2" rpy="0 0 0"/>
     <!-- 회전축 -->
-    <axis xyz="0 1 0"/>
+    <axis xyz="0 -1 0"/>
     <!-- 임시 limit -->
-    <limit lower="-1.57" upper="1.57" effort="1" velocity="1"/>
+    <limit lower="0" upper="3.14" effort="1" velocity="1"/>
   </joint>
   <!-- gripper base -->
@@ -71,5 +71,5 @@
     </visual>
   </link>
-  <!-- joint3: link2 -> gripper base -->
+  <!-- joint4: link2 -> gripper base -->
   <joint name="joint4" type="revolute">
     <parent link="link2"/>
@@ -79,5 +79,5 @@
     <axis xyz="0 0 1"/>
     <!-- 임시 limit -->
-    <limit lower="-1.57" upper="1.57" effort="1" velocity="1"/>
+    <limit lower="0" upper="3.14" effort="1" velocity="1"/>
   </joint>
   <!-- gripper left 1 -->
@@ -92,9 +92,9 @@
     <parent link="gripper_base"/>
     <child link="gripper_left_1"/>
-    <origin xyz="0.0051 0.0105 0.029" rpy="0 0 0"/>
+    <origin xyz="0.0051 0.0105 0.029" rpy="1.57 0 0"/>
     <!-- 이동축 -->
-    <axis xyz="1 0 0"/>
+    <axis xyz="-1 0 0"/>
     <!-- 임시 limit -->
-    <limit lower="-1.57" upper="0" effort="1" velocity="0.02"/>
+    <limit lower="1.57" upper="3.14" effort="1" velocity="0.02"/>
   </joint>
   <!-- gripper right 1 -->
@@ -109,9 +109,9 @@
     <parent link="gripper_base"/>
     <child link="gripper_right_1"/>
-    <origin xyz="0.0051 -0.0105 0.029" rpy="0 0 0"/>
+    <origin xyz="0.0051 -0.0105 0.029" rpy="-1.57 0 0"/>
     <!-- 이동축 -->
-    <axis xyz="1 0 0"/>
+    <axis xyz="-1 0 0"/>
     <!-- 임시 limit -->
-    <limit lower="-1.57" upper="0" effort="1" velocity="0.02"/>
+    <limit lower="1.57" upper="3.14" effort="1" velocity="0.02"/>
     <!-- 왼쪽 그리퍼와 반대 방향으로 연동 -->
     <mimic joint="gripper_left_joint_1" multiplier="-1" offset="0"/>
